File: pcb_challenge_final.kicad_sch (KiCad schematic)
At the start: 164 parts, among them J4 Conn_01x04_Pin, J5 Conn_01x04_Pin, Q12 Q_Dual_NPN_PNP_B1E2B2C2E1C1, Q13 Q_Dual_NPN_PNP_B1E2B2C2E1C1, Q14 Q_Dual_NPN_PNP_B1E2B2C2E1C1, Q15 Q_Dual_NPN_PNP_B1E2B2C2E1C1, Q16 Q_Dual_NPN_PNP_B1E2B2C2E1C1, Q18 Q_Dual_NPN_PNP_B1E2B2C2E1C1, Q19 Q_Dual_NPN_PNP_B1E2B2C2E1C1, Q20 Q_Dual_NPN_PNP_B1E2B2C2E1C1, Q21 Q_Dual_NPN_PNP_B1E2B2C2E1C1, Q22 Q_Dual_NPN_PNP_B1E2B2C2E1C1, Q23 Q_Dual_NPN_PNP_B1E2B2C2E1C1, Q24 Q_Dual_NPN_PNP_B1E2B2C2E1C1, Q25 Q_Dual_NPN_PNP_B1E2B2C2E1C1, Q26 Q_Dual_NPN_PNP_B1E2B2C2E1C1, Q27 Q_Dual_NPN_PNP_B1E2B2C2E1C1, SW1 SW_Push, SW2 SW_MEC_5G, SW3 SW_Push, U1 74AUP1G80, U10 NMUX1308BQ, U11 NMUX1308BQ, U12 NMUX1308BQ, U13 NMUX1308BQ, U14 NMUX1308BQ, U15 NMUX1308BQ, U16 NMUX1308BQ, U17 74AUP1G80, U18 74AHC1G86, U19 74AUP1G80, U20 74AUP1G80, U21 74LV1T08GV, U22 CD74HC283M96, U23 74LV1T08GV, U24 74LVC1GU04DRL, U25 ESP32-S3-MINI-1, U26 74LVC1GU04DRL, U27 74LV1T08GV, U28 CD74HC283M96, U29 NMUX1308BQ, U3 74AHC1G86, U30 NMUX1308BQ, U31 NMUX1308BQ, U32 NMUX1308BQ, U33 74AUP1G80, U34 74AUP1G80, U35 NMUX1308BQ, U36 NMUX1308BQ, U37 74AUP1G80, U38 74AUP1G80, U39 NMUX1308BQ, U4 74AUP1G80, U40 NMUX1308BQ, U41 NMUX1308BQ, U42 NMUX1308BQ, U43 NMUX1308BQ, U44 NMUX1308BQ, U45 74AUP1G80, U46 74AUP1G80, U47 74AUP1G80, U48 74AUP1G80, U49 74AUP1G80, U5 74AUP1G80, U50 74AUP1G80, U51 74LV1T08GV, U52 74AHC1G86, U53 74LVC1GU04DRL, U54 74LVC1GU04DRL, U55 74AHC1G86, U56 74AHC1G86, U57 74LVC1GU04DRL, U58 74LVC1GU04DRL, U59 74LV1T08GV, U6 74AUP1G80, U60 74AHC1G86, U61 74LVC1GU04DRL, U62 74LV1T08GV, U63 74LV1T08GV, U64 NMUX1308BQ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

Commit message: Save current four-layer layout and remaining work
Parts:
- removed Q12, Q13, Q14: Q_Dual_NPN_PNP_B1E2B2C2E1C1, Package_TO_SOT_SMD:SOT-1123, symbol Transistor_BJT:Q_Dual_NPN_PNP_B1E2B2C2E1C1
- added Q17, Q28, Q29: Q_Dual_NPN_PNP_B1E2B2C2E1C1, Package_TO_SOT_SMD:SOT-1123, symbol Transistor_BJT:Q_Dual_NPN_PNP_B1E2B2C2E1C1
- C1, C2, C3, C4, C5, C6, C7, C8: footprint (none) -> Capacitor_SMD:C_0201_0603Metric
- R1: footprint (none) -> Capacitor_SMD:C_0402_1005Metric
- SW1, SW3: footprint (none) -> Button_Switch_SMD:SW_DIP_SPSTx01_Slide_6.7x4.1mm_W8.61mm_P2.54mm_LowProfile
Connections:
- net 3v3 is gone; now on net +3.3V: C1.1, C2.1, R1.1, U25.3 (3V3)
- net CLK is gone; now on net clk: R7.2, Y2.3 (CLK)
- net b1: now also Q29.2 (C1)
- net b2: now also Q28.2 (C1)
- net b3: now also Q17.2 (C1)
- net b4: now also Q15.2 (C1)
- net rst: now also Q17.1 (B1), Q28.1 (B1), Q29.1 (B1)
- net rw1: now also Q20.2 (C1); no longer Q18.6 (C1)
- net rw2: now also Q19.2 (C1); no longer Q19.6 (C1)
- net rw3: now also Q18.2 (C1); no longer Q20.6 (C1)
- net wr1: now also Q23.2 (C1); no longer Q23.6 (C1)
- net wr2: now also Q22.2 (C1); no longer Q22.6 (C1)
- net wr3: now also Q21.2 (C1); no longer Q21.6 (C1)
- net at R62.2: now also Q24.3 (E1); no longer Q24.5 (E1)
- net at R36.2: now also Q20.3 (E1); no longer Q18.5 (E1)
- net at R44.2: now also Q21.3 (E1); no longer Q21.5 (E1)
- net at R64.2: now also Q25.3 (E1); no longer Q25.5 (E1)
- net at U67.1 (D), U71.4 (Out): now also Q25.2 (C1); no longer Q25.6 (C1)
- net at R66.2: now also Q26.3 (E1); no longer Q26.5 (E1)
- net at R28.2: now also Q17.3 (E1)
- net at U66.1 (D), U72.4 (Out): now also Q24.2 (C1); no longer Q24.6 (C1)
- net at R22.2: now also Q29.3 (E1)
- net at R45.2: now also Q22.3 (E1); no longer Q22.5 (E1)
- net at R30.2: now also Q15.3 (E1); no longer Q15.5 (E1)
- net at U68.1 (D), U70.4 (Out): now also Q26.2 (C1); no longer Q26.6 (C1)
- net at R32.2: now also Q16.3 (E1); no longer Q16.5 (E1)
- net at R26.2: now also Q28.3 (E1)
- net at U69.1 (D), U73.4 (Out): now also Q27.2 (C1); no longer Q27.6 (C1)
- net at R40.2: now also Q18.3 (E1); no longer Q20.5 (E1)
- net at U1.1 (D), U27.4 (Y): now also Q16.2 (C1); no longer Q16.6 (C1)
- net at R38.2: now also Q19.3 (E1); no longer Q19.5 (E1)
- net at R46.2: now also Q23.3 (E1); no longer Q23.5 (E1)
- net at R68.2: now also Q27.3 (E1); no longer Q27.5 (E1)
- removed net Input 4: Q15.6 (C1)
