File: pcb_challenge_final.kicad_pcb (KiCad board)
At the start: 2 copper layers, 154 parts, among them J4 Conn_01x04_Pin, J5 Conn_01x04_Pin, Q12 Q_Dual_NPN_PNP_B1E2B2C2E1C1, Q13 Q_Dual_NPN_PNP_B1E2B2C2E1C1, Q14 Q_Dual_NPN_PNP_B1E2B2C2E1C1, Q15 Q_Dual_NPN_PNP_B1E2B2C2E1C1, Q16 Q_Dual_NPN_PNP_B1E2B2C2E1C1, Q18 Q_Dual_NPN_PNP_B1E2B2C2E1C1, Q19 Q_Dual_NPN_PNP_B1E2B2C2E1C1, Q20 Q_Dual_NPN_PNP_B1E2B2C2E1C1, Q21 Q_Dual_NPN_PNP_B1E2B2C2E1C1, Q22 Q_Dual_NPN_PNP_B1E2B2C2E1C1, Q23 Q_Dual_NPN_PNP_B1E2B2C2E1C1, Q24 Q_Dual_NPN_PNP_B1E2B2C2E1C1, Q25 Q_Dual_NPN_PNP_B1E2B2C2E1C1, Q26 Q_Dual_NPN_PNP_B1E2B2C2E1C1, Q27 Q_Dual_NPN_PNP_B1E2B2C2E1C1, SW2 SW_MEC_5G, U1 74AUP1G80, U10 NMUX1308BQ, U11 NMUX1308BQ, U12 NMUX1308BQ, U13 NMUX1308BQ, U14 NMUX1308BQ, U15 NMUX1308BQ, U16 NMUX1308BQ, U17 74AUP1G80, U18 74AHC1G86, U19 74AUP1G80, U2 NMUX1308BQ, U20 74AUP1G80, U21 74LV1T08GV, U22 CD74HC283M96, U23 74LV1T08GV, U24 74LVC1GU04DRL, U25 ESP32-S3-MINI-1, U26 74LVC1GU04DRL, U27 74LV1T08GV, U28 CD74HC283M96, U29 NMUX1308BQ, U3 74AHC1G86, U30 NMUX1308BQ, U31 NMUX1308BQ, U32 NMUX1308BQ, U33 74AUP1G80, U34 74AUP1G80, U35 NMUX1308BQ, U36 NMUX1308BQ, U37 74AUP1G80, U38 74AUP1G80, U39 NMUX1308BQ, U4 74AUP1G80, U40 NMUX1308BQ, U41 NMUX1308BQ, U42 NMUX1308BQ, U43 NMUX1308BQ, U44 NMUX1308BQ, U45 74AUP1G80, U46 74AUP1G80, U47 74AUP1G80, U48 74AUP1G80, U49 74AUP1G80, U5 74AUP1G80, U50 74AUP1G80, U51 74LV1T08GV, U52 74AHC1G86, U53 74LVC1GU04DRL, U54 74LVC1GU04DRL, U55 74AHC1G86, U56 74AHC1G86, U57 74LVC1GU04DRL, U58 74LVC1GU04DRL, U59 74LV1T08GV, U6 74AUP1G80, U60 74AHC1G86, U61 74LVC1GU04DRL, U62 74LV1T08GV, U63 74LV1T08GV, U64 NMUX1308BQ, U65 74AUP1G80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

Commit message: Save current four-layer layout and remaining work
Parts:
- removed Q12, Q13, Q14: Q_Dual_NPN_PNP_B1E2B2C2E1C1, Package_TO_SOT_SMD:SOT-1123
- removed U2: NMUX1308BQ, Package_DFN_QFN:DHVQFN-16-1EP_2.5x3.5mm_P0.5mm_EP1x2mm
- added C1: 22uF, Capacitor_SMD:C_0201_0603Metric, F.Cu at (102.5, 103.0)
- added C2: 0.1uF, Capacitor_SMD:C_0201_0603Metric, F.Cu at (102.5, 104.3)
- added C3: 12pF, Capacitor_SMD:C_0201_0603Metric, F.Cu at (110.0, 116.5)
- added C4: 12pF, Capacitor_SMD:C_0201_0603Metric, F.Cu at (110.0, 115.4)
- added C5: 22pF, Capacitor_SMD:C_0201_0603Metric, F.Cu at (109.5, 121.8)
- added C6: 22pF, Capacitor_SMD:C_0201_0603Metric, F.Cu at (111.1, 121.8)
- added C7: 22uF, Capacitor_SMD:C_0201_0603Metric, F.Cu at (124.0, 101.5)
- added C8: 0.1uF, Capacitor_SMD:C_0201_0603Metric, F.Cu at (124.0, 102.8)
- added Q17: Q_Dual_NPN_PNP_B1E2B2C2E1C1, Package_TO_SOT_SMD:SOT-1123, F.Cu at (159.4, 159.4)
- added Q28: Q_Dual_NPN_PNP_B1E2B2C2E1C1, Package_TO_SOT_SMD:SOT-1123, F.Cu at (159.4, 162.0)
- added Q29: Q_Dual_NPN_PNP_B1E2B2C2E1C1, Package_TO_SOT_SMD:SOT-1123, F.Cu at (159.4, 164.6)
- added R1: 10k, Capacitor_SMD:C_0402_1005Metric, F.Cu at (125.2, 104.5)
- added SW1: SW_Push, Button_Switch_SMD:SW_DIP_SPSTx01_Slide_6.7x4.1mm_W8.61mm_P2.54mm_LowProfile, F.Cu at (135.0, 102.5)
- added SW3: SW_Push, Button_Switch_SMD:SW_DIP_SPSTx01_Slide_6.7x4.1mm_W8.61mm_P2.54mm_LowProfile, F.Cu at (147.0, 102.5)
- R21, R22, R23, R25, R26, R27, R28, R29, R30, R31, R32, R33, R34, R35, R36, R37, R38, R39, R40, R41, R42, R43, R44, R45, R46, R47, R48, R49, R50, R51, R52, R53, R54, R55, R56, R57, R58, R59, R61, R62, R63, R64, R65, R66, R67, R68: moved to B.Cu
- SW2: value SW_MEC_5G -> SW_Push; footprint Button_Switch_SMD:SW_SPST_CK_RS282G05A3 -> Button_Switch_SMD:SW_DIP_SPSTx01_Slide_6.7x4.1mm_W8.61mm_P2.54mm_LowProfile
- moved J5 74.1 mm to (102.0, 134.0)
- moved J3 73.6 mm to (104.0, 120.6), turned to -90 degrees
- moved Y2 72.3 mm to (106.8, 129.0)
- moved U54 69.4 mm to (106.0, 163.5)
- moved U57 66.2 mm to (114.8, 163.5)
- moved U53 65.6 mm to (110.4, 163.5)
- moved D1 62.5 mm to (121.5, 112.0), turned to 90 degrees
- moved R15 61.5 mm to (114.0, 124.0), turned to 90 degrees
- moved U58 61.1 mm to (119.2, 163.5)
- moved R20 59.3 mm to (117.0, 124.0), turned to 90 degrees
- moved Q16 57.1 mm to (147.5, 159.3)
- moved U61 56.1 mm to (123.6, 163.5)
- moved Q15 53.8 mm to (159.4, 156.8)
- moved U29 52.2 mm to (111.0, 137.0)
- moved U31 52.0 mm to (111.0, 143.0)
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Connections:
- C9 pad 1: NRST -> rst
- J3 pad SH: (no net) -> Net-(J3-SHIELD)
- Q15 pad 2: (no net) -> b4
- Q15 pad 3: (no net) -> Net-(Q15A-E1)
- Q16 pad 2: (no net) -> Net-(Q16A-C1)
- Q16 pad 3: (no net) -> Net-(Q16A-E1)
- Q18 pad 2: (no net) -> rw3
- Q18 pad 3: (no net) -> Net-(Q18A-E1)
- Q19 pad 2: (no net) -> rw2
- Q19 pad 3: (no net) -> Net-(Q19A-E1)
- Q20 pad 2: (no net) -> rw1
- Q20 pad 3: (no net) -> Net-(Q20A-E1)
- Q21 pad 2: (no net) -> wr3
- Q21 pad 3: (no net) -> Net-(Q21A-E1)
- Q22 pad 2: (no net) -> wr2
- Q22 pad 3: (no net) -> Net-(Q22A-E1)
- Q23 pad 2: (no net) -> wr1
- Q23 pad 3: (no net) -> Net-(Q23A-E1)
- Q24 pad 2: (no net) -> Net-(Q24A-C1)
- Q24 pad 3: (no net) -> Net-(Q24A-E1)
- Q25 pad 2: (no net) -> Net-(Q25A-C1)
- Q25 pad 3: (no net) -> Net-(Q25A-E1)
- Q26 pad 2: (no net) -> Net-(Q26A-C1)
- Q26 pad 3: (no net) -> Net-(Q26A-E1)
- Q27 pad 2: (no net) -> Net-(Q27A-C1)
- Q27 pad 3: (no net) -> Net-(Q27A-E1)
- R36 pad 2: Net-(Q18A-E1) -> Net-(Q20A-E1)
- R40 pad 2: Net-(Q20A-E1) -> Net-(Q18A-E1)
- R7 pad 2: CLK -> clk
- SW2 pad 2: GND -> rst
- U25 pad 3: 3v3 -> +3.3V
- Y2 pad 3: CLK -> clk
Routing:
- net IO8: track 0.00 -> 270.7 mm, vias 0 -> 19
- net IO6: track 0.00 -> 252.6 mm, vias 0 -> 19
- net rst: track 0.00 -> 243.8 mm, vias 0 -> 17
- net GND: track 0.00 -> 213.8 mm, vias 0 -> 141
- net clk: track 0.00 -> 181.8 mm, vias 0 -> 15
- net IO9: track 0.00 -> 119.2 mm, vias 0 -> 5
- net +3.3V: track 0.00 -> 111.4 mm, vias 0 -> 81
- net +5V: track 0.00 -> 91.0 mm, vias 0 -> 4
- net ???: track 0.00 -> 86.9 mm, vias 0 -> 2
- net wir1: track 0.00 -> 60.7 mm, vias 0 -> 4
- net Net-(U25-IO0): track 0.00 -> 44.3 mm, vias 0 -> 2
- net COUT: track 0.00 -> 44.0 mm, vias 0 -> 3
- net Net-(U25-EN): track 0.00 -> 37.0 mm, vias 0 -> 4
- net reg1: track 0.00 -> 35.8 mm, vias 0 -> 2
- net ws2: track 0.00 -> 31.9 mm, vias 0 -> 3
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- added copper zone on In2.Cu, net +3.3V
- added copper zone on In1.Cu, net GND
- added copper zone on F.Cu, net Net-(U25-GND-Pad2)
Other:
- board outline added: 66.7 x 67.2 mm
- copper layers 2 -> 4

Commit message: Save routing progress with 18 connections remaining
Routing:
- net IO10: track 7.61 -> 144.3 mm, vias 2 -> 3
- net IO11: track 7.61 -> 139.4 mm, vias 2 -> 3
- net IO12: track 7.61 -> 134.6 mm, vias 2 -> 3
- net IO13: track 7.61 -> 130.9 mm, vias 2 -> 3
- net r_en: track 1.69 -> 106.3 mm, vias 1 -> 13
- net b1: track 0.00 -> 84.1 mm, vias 0 -> 1
- net b3: track 0.00 -> 79.3 mm, vias 0 -> 2
- net b2: track 0.00 -> 79.1 mm, vias 0 -> 2
- net b4: track 0.00 -> 78.0 mm, vias 0 -> 3
- net rc1: track 7.08 -> 76.9 mm, vias 3 -> 7
- net R_en: track 1.69 -> 59.5 mm, vias 1 -> 8
- net out_1: track 0.00 -> 57.7 mm, vias 0 -> 6
- net out_2: track 0.00 -> 52.7 mm, vias 0 -> 2
- net out_3: track 0.00 -> 42.0 mm
- net rw3: track 2.62 -> 42.2 mm
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